File: PCB/fechadura_eletronica/fechadura_eletronica_vFinal.kicad_pcb (KiCad board)
At the start: 2 copper layers, 73 x 77 mm, 21 parts, among them J1 Relay Module, J2 RFID - RC522, J3 LCD 16X2, J4 DY50, SW1 reset button, U1 LM7805 - regulator, U2 ESP32-DEVKIT-V1, U3 LD1117S33TR_SOT223

Commit message: versao final
Parts:
- moved BZ1 3.31 mm to (142.8, 100.0)
Routing:
- net +5V: track 18.3 -> 43.3 mm
- net Net-(U2-D26): track 70.3 -> 66.2 mm
- net Net-(BZ1-+): track 35.3 -> 31.9 mm
Other:
- board size 73 x 77 mm -> 80 x 80 mm
Changed lines of the file:
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@@
 	(footprint "Buzzer_Beeper:Buzzer_12x9.5RM7.6"
 		(layer "F.Cu")
-		(at 142.6 103.3 180)
+		(at 142.8 100 180)
 		(descr "Generic Buzzer, D12mm height 9.5mm with RM7.6mm")
 		(tags "buzzer")
@@
 	(gr_line
 		(start 75 112)
-		(end 148.000394 112)
+		(end 155 112)
 		(stroke
 			(width 0.7)
@@
 	(gr_line
 		(start 75 112)
-		(end 75 35)
+		(end 75 32)
 		(stroke
 			(width 0.7)
@@
 	)
 	(gr_line
-		(start 75 35)
-		(end 148.001667 35)
+		(start 75 32)
+		(end 155 32)
 		(stroke
 			(width 0.7)
@@
 	)
 	(gr_line
-		(start 148.001667 35)
-		(end 148.000394 112)
+		(start 155 32)
+		(end 154.998604 112)
 		(stroke
 			(width 0.7)
@@
 	)
 	(segment
-		(start 143 73.63)
-		(end 140.7 71.33)
+		(start 140.7 71.33)
+		(end 138.47 71.33)
 		(width 0.7)
 		(layer "B.Cu")
@@
 	)
 	(segment
-		(start 143 102.9)
-		(end 143 73.63)
+		(start 143 73.63)
+		(end 140.7 71.33)
 		(width 0.7)
 		(layer "B.Cu")
@@
 	)
 	(segment
-		(start 140.7 71.33)
-		(end 138.47 71.33)
+		(start 143 99.8)
+		(end 143 73.63)
 		(width 0.7)
 		(layer "B.Cu")
@@
 	)
 	(segment
-		(start 142.6 103.3)
-		(end 143 102.9)
+		(start 142.8 100)
+		(end 143 99.8)
 		(width 0.7)
 		(layer "B.Cu")
@@
 	)
 	(segment
-		(start 138.47 66.25)
-		(end 141.94 66.25)
+		(start 105.5 39)
+		(end 105.25 38.75)
 		(width 0.7)
 		(layer "B.Cu")
@@
 	)
 	(segment
-		(start 144.45 42.45)
-		(end 141 39)
+		(start 134 39)
+		(end 105.5 39)
 		(width 0.7)
 		(layer "B.Cu")
@@
 	)
 	(segment
-		(start 144.45 65.55)
-		(end 144.45 42.45)
+		(start 138.47 66.25)
+		(end 141.94 66.25)
 		(width 0.7)
 		(layer "B.Cu")
@@
 	)
 	(segment
-		(start 142 66.31)
-		(end 143.69 66.31)
+		(start 144.45 49.45)
+		(end 134 39)
 		(width 0.7)
 		(layer "B.Cu")
@@
 	)
 	(segment
-		(start 105.5 39)
-		(end 105.25 38.75)
+		(start 142 66.31)
+		(end 143.69 66.31)
 		(width 0.7)
 		(layer "B.Cu")
@@
 	)
 	(segment
-		(start 144.45 65.57)
-		(end 144.45 65.55)
+		(start 144.45 65.55)
+		(end 144.45 49.45)
 		(width 0.7)
 		(layer "B.Cu")
@@
 	)
 	(segment
-		(start 141 39)
-		(end 105.5 39)
+		(start 144.45 65.57)
+		(end 144.45 65.55)
 		(width 0.7)
 		(layer "B.Cu")
@@
 	)
 	(segment
+		(start 113.5 100)
+		(end 113.5 103)
+		(width 0.9)
+		(layer "B.Cu")
+		(net 28)
+	)
+	(segment
+		(start 96.5 97.5)
+		(end 98 99)
+		(width 0.9)
+		(layer "B.Cu")
+		(net 28)
+	)
+	(segment
 		(start 89.475 88.5)
 		(end 89.46 88.515)
@@
 		(width 0.9)
 		(layer "B.Cu")
+		(net 28)
+	)
+	(segment
+		(start 98 99)
+		(end 112.5 99)
+		(width 0.9)
+		(layer "B.Cu")
+		(net 28)
+	)
+	(segment
+		(start 112.5 99)
+		(end 113.5 100)
+		(width 0.9)
+		(layer "B.Cu")
+		(net 28)
+	)
+	(segment
+		(start 92.5 97.5)
+		(end 96.5 97.5)
+		(width 0.9)
+		(layer "B.Cu")
